Commit message: Odom: Experiment with finding theta. Velocity calcs still waaay off..

File: urdf/oskar.urdf (robot description, URDF)
Before this commit: robot Oskar III, 3 links, 2 joints
Joints:
- joint left_wheel_to_base: origin xyz=0.1075 -0.1851 -0.05 rpy=1.57 0.0 0.0 -> xyz=0.1075 0.1851 -0.05 rpy=1.57 0.0 0.0
- joint right_wheel_to_base: origin xyz=0.1075 0.1851 -0.05 rpy=1.57 0.0 0.0 -> xyz=0.1075 -0.1851 -0.05 rpy=1.57 0.0 0.0

Commit message: Odom: speeds equalized

File: urdf/oskar.urdf (robot description, URDF)
Before this commit: robot Oskar III, 3 links, 2 joints
Joints:
- joint left_wheel_to_base: child left_wheel -> right_wheel; origin xyz=0.1075 0.1851 -0.05 rpy=1.57 0.0 0.0 -> xyz=0.1075 -0.1851 -0.05 rpy=1.57 0.0 0.0
- joint right_wheel_to_base: child right_wheel -> left_wheel; origin xyz=0.1075 -0.1851 -0.05 rpy=1.57 0.0 0.0 -> xyz=0.1075 0.1851 -0.05 rpy=1.57 0.0 0.0

Commit message: General: add parameter server MotorPlugin: Write speed calculation to be more explicit

File: urdf/oskar.urdf (robot description, URDF)
Before this commit: robot Oskar III, 3 links, 2 joints
Links:
- link left_wheel: geometry visual cylinder length=0.05 radius=0.075
- link right_wheel: geometry visual cylinder length=0.05 radius=0.075

Commit message: Remove unused debug statements from odom plugin. Add joints and upper body to urdf

File: urdf/oskar.urdf (robot description, URDF)
Before this commit: robot Oskar III, 3 links, 2 joints
Links:
- added link oskar3_body; visual cylinder length=1.5 radius=0.5
Joints:
- added joint oskar3_body_tilt: type revolute, parent base_link, child oskar3_body, origin xyz=0.215 0 0.540, axis 0 1 0, limit lower=0.140 upper=1.0 effort=0.0 velocity=0.0
- added joint oskar3_body_to_base: type prismatic, parent base_link, child oskar3_body, origin xyz=0.215 0 0.140, axis 0 0 1, limit lower=0.140 upper=1.0 effort=0.0 velocity=0.0

Commit message: URDF changes. Attempt to ignore usb conn for viz. No success

File: urdf/oskar.urdf (robot description, URDF)
Before this commit: robot Oskar III, 4 links, 4 joints
Links:
- removed link oskar3_body
- added link body; visual cylinder length=1.5 radius=0.5
- added link body_mountpoint; visual box size=0.01 0.01 0.01
- added link left_elbow; visual box size=0.1 0.1 0.1
- added link left_forearm; visual cylinder length=0.5 radius=0.1
- added link left_shoulder; visual box size=0.1 0.1 0.1
- added link left_upper_arm; visual cylinder length=.5 radius=0.1
- added link left_upper_arm_rotational; visual box size=0.1 0.1 0.1
- added link right_elbow; visual box size=0.1 0.1 0.1
- added link right_forearm; visual cylinder length=0.5 radius=0.1
- added link right_shoulder; visual box size=0.1 0.1 0.1
- added link right_upper_arm; visual cylinder length=.5 radius=0.1
- added link right_upper_arm_rotational; visual box size=0.1 0.1 0.1
Joints:
- removed joint oskar3_body_tilt
- removed joint oskar3_body_to_base
- added joint bowing_joint: type revolute, parent body_mountpoint, child body, origin xyz=0.0 0.0 0.0 rpy=0.0 0.0 0.0, axis 0 1 0, limit lower=0 upper=1.0 effort=0.0 velocity=0.0
- added joint kneeling_joint: type prismatic, parent base_link, child body_mountpoint, origin xyz=0 0 0.07, axis 0.0 0.0 1.0, limit lower=0 upper=1 effort=0.0 velocity=0.0
- added joint left_elbow_joint: type revolute, parent left_upper_arm, child left_elbow, origin xyz=0.0 0.0 -0.25 rpy=0.0 0.0 0.0, axis 0 -1.0 0.0, limit lower=0.0 upper=1.0 effort=0.0 velocity=0.0
- added joint left_forearm_to_elbow: type fixed, parent left_elbow, child left_forearm, origin xyz=0.0 0.0 -0.25 rpy=0.0 0.0 0.0
- added joint left_shoulder_to_body: type revolute, parent body, child left_shoulder, origin xyz=0.0 0.6 .65 rpy=0.0 0.0 0.0, axis 0.0 1 0.0, limit lower=-1.0 upper=1.0 effort=0.0 velocity=0.0
- added joint left_upper_arm_to_left_shoulder: type revolute, parent left_shoulder, child left_upper_arm_rotational, origin xyz=0.0 0.0 0 rpy=0.0 0.0 0.0, axis 1.0 0.0 0.0, limit lower=0.0 upper=1.0 effort=0.0 velocity=0.0
- added joint left_upper_arm_to_shoulder_joints: type fixed, parent left_upper_arm_rotational, child left_upper_arm, origin xyz=0.0 0.0 -0.25 rpy=0.0 0.0 0.0
- added joint right_elbow_joint: type revolute, parent right_upper_arm, child right_elbow, origin xyz=0.0 0.0 -0.25 rpy=0.0 0.0 0.0, axis 0.0 -1.0 0.0, limit lower=0.0 upper=1.0 effort=0.0 velocity=0.0
- added joint right_forearm_to_elbow: type fixed, parent right_elbow, child right_forearm, origin xyz=0.0 0.0 -0.25 rpy=0.0 0.0 0.0
- added joint right_shoulder_to_body: type revolute, parent body, child right_shoulder, origin xyz=0.0 -0.6 .65 rpy=0.0 0.0 0.0, axis 0.0 1 0.0, limit lower=-1.0 upper=1.0 effort=0.0 velocity=0.0
- added joint right_upper_arm_to_right_shoulder: type revolute, parent right_shoulder, child right_upper_arm_rotational, origin xyz=0.0 0.0 0 rpy=0.0 0.0 0.0, axis -1.0 0.0 0.0, limit lower=0.0 upper=1.0 effort=0.0 velocity=0.0
- added joint right_upper_arm_to_shoulder_joints: type fixed, parent right_upper_arm_rotational, child right_upper_arm, origin xyz=0.0 0.0 -0.25 rpy=0.0 0.0 0.0

Commit message: URDF actual dimensions and limits

File: urdf/oskar.urdf (robot description, URDF)
Before this commit: robot Oskar III, 15 links, 14 joints
Links:
- added link body_mountpoint2; visual box size=0.01 0.01 0.01
- link base_link: geometry visual box size=0.600 0.600 0.300
- link body: geometry visual cylinder length=0.560 radius=0.250
- link left_elbow: geometry visual box size=0.01 0.01 0.01
- link left_forearm: geometry visual cylinder length=.330 radius=0.01685
- link left_upper_arm: geometry visual cylinder length=.330 radius=0.01685
- link left_wheel: geometry visual cylinder length=0.045 radius=0.075
- link right_elbow: geometry visual box size=0.01 0.01 0.01
- link right_forearm: geometry visual cylinder length=.330 radius=0.01685
- link right_upper_arm: geometry visual cylinder length=.330 radius=0.01685
- link right_wheel: geometry visual cylinder length=0.045 radius=0.075
Joints:
- added joint body_to_mount: type fixed, parent body_mountpoint2, child body, origin xyz=0.0 0.0 0.080 rpy=0.0 0.0 0.0
- joint bowing_joint: child body -> body_mountpoint2; limit lower=0 upper=1.0 effort=0.0 velocity=0.0 -> lower=0 upper=0.4 effort=0.0 velocity=0.0
- joint kneeling_joint: limit lower=0 upper=1 effort=0.0 velocity=0.0 -> lower=0.620 upper=0.950 effort=0.0 velocity=0.0; origin xyz=0 0 0.07 -> xyz=0 0 0.0860
- joint left_elbow_joint: limit lower=0.0 upper=1.0 effort=0.0 velocity=0.0 -> lower=0.0 upper=2.04 effort=0.0 velocity=0.0; origin xyz=0.0 0.0 -0.25 rpy=0.0 0.0 0.0 -> xyz=0.0 0.0 -0.165  rpy=0.0 0.0 0.0
- joint left_forearm_to_elbow: origin xyz=0.0 0.0 -0.25 rpy=0.0 0.0 0.0 -> xyz=0.0 0.0 -0.165 rpy=0.0 0.0 0.0
- joint left_shoulder_to_body: limit lower=-1.0 upper=1.0 effort=0.0 velocity=0.0 -> lower=-3.14 upper=0 effort=0.0 velocity=0.0; origin xyz=0.0 0.6 .65 rpy=0.0 0.0 0.0 -> xyz=0 0.317 0.213 rpy=0.0 0.0 0.0
- joint left_upper_arm_to_left_shoulder: limit lower=0.0 upper=1.0 effort=0.0 velocity=0.0 -> lower=0.0 upper=3.14 effort=0.0 velocity=0.0
- joint left_upper_arm_to_shoulder_joints: origin xyz=0.0 0.0 -0.25 rpy=0.0 0.0 0.0 -> xyz=0.0 0.0 -0.165 rpy=0.0 0.0 0.0
- joint left_wheel_to_base: origin xyz=0.1075 -0.1851 -0.05 rpy=1.57 0.0 0.0 -> xyz=0.214 -0.240 -0.110 rpy=1.57 0.0 0.0
- joint right_elbow_joint: limit lower=0.0 upper=1.0 effort=0.0 velocity=0.0 -> lower=0.0 upper=2.04 effort=0.0 velocity=0.0; origin xyz=0.0 0.0 -0.25 rpy=0.0 0.0 0.0 -> xyz=0.0 0.0 -0.165 rpy=0.0 0.0 0.0
- joint right_forearm_to_elbow: origin xyz=0.0 0.0 -0.25 rpy=0.0 0.0 0.0 -> xyz=0.0 0.0 -0.165 rpy=0.0 0.0 0.0
- joint right_shoulder_to_body: limit lower=-1.0 upper=1.0 effort=0.0 velocity=0.0 -> lower=-3.14 upper=0 effort=0.0 velocity=0.0; origin xyz=0.0 -0.6 .65 rpy=0.0 0.0 0.0 -> xyz=0 -0.317 0.213 rpy=0.0 0 0.0
- joint right_upper_arm_to_right_shoulder: limit lower=0.0 upper=1.0 effort=0.0 velocity=0.0 -> lower=0.0 upper=3.14 effort=0.0 velocity=0.0
- joint right_upper_arm_to_shoulder_joints: origin xyz=0.0 0.0 -0.25 rpy=0.0 0.0 0.0 -> xyz=0.0 0.0 -0.165 rpy=0.0 0.0 0.0
- joint right_wheel_to_base: origin xyz=0.1075 0.1851 -0.05 rpy=1.57 0.0 0.0 -> xyz=0.214 0.240 -0.110 rpy=1.57 0.0 0.0

Commit message: Implementmore compact format instructions from ROS, also try moveit

File: urdf/oskar.urdf (robot description, URDF)
Before this commit: robot Oskar III, 16 links, 15 joints
Links:
- added link left_gripper; visual box size=0.1 0.1 0.1
- added link right_gripper; visual box size=0.1 0.1 0.1
- link left_shoulder: geometry visual box size=0.01 0.01 0.01
- link left_upper_arm_rotational: geometry visual box size=0.01 0.01 0.01
- link right_shoulder: geometry visual box size=0.01 0.01 0.01
- link right_upper_arm_rotational: geometry visual box size=0.01 0.01 0.01
Joints:
- added joint left_ripper_to_right_forearm: type fixed, parent left_forearm, child left_gripper, origin xyz=0.0 0.0 -0.165 rpy=0.0 0.0 0.0
- added joint right_ripper_to_right_forearm: type fixed, parent right_forearm, child right_gripper, origin xyz=0.0 0.0 -0.165 rpy=0.0 0.0 0.0
